Commit message: Update steering limits in URDF to allow for full rotation (±180 degrees)

File: ackerman_description/urdf/fw-max.xacro (robot description, xacro)
@@ -49,5 +49,5 @@
         <origin xyz="0.3 0.225 0" />
         <axis xyz="0 0 1" />
-        <limit lower="-1.57" upper="1.57" effort="50.0" velocity="50.0"/>
+        <limit lower="-3.14" upper="3.14" effort="50.0" velocity="50.0"/>
     </joint>
     <transmission name="left_steering_hinge_trans">
@@ -105,5 +105,5 @@
         <origin xyz="0.3 -0.225 0" />
         <axis xyz="0 0 1" />
-        <limit lower="-1.57" upper="1.57" effort="50.0" velocity="50.0"/>
+        <limit lower="-3.14" upper="3.14" effort="50.0" velocity="50.0"/>
         <mimic joint="left_steering_hinge_joint" multiplier="1.0" offset="0.0"/>
     </joint>
@@ -161,5 +161,5 @@
         <origin xyz="-0.3 0.225 0" />
         <axis xyz="0 0 1" />
-        <limit lower="-1.57" upper="1.57" effort="50.0" velocity="50.0"/>
+        <limit lower="-3.14" upper="3.14" effort="50.0" velocity="50.0"/>
         <mimic joint="left_steering_hinge_joint" multiplier="-1.0" offset="0.0"/>
     </joint>
@@ -217,5 +217,5 @@
         <origin xyz="-0.3 -0.225 0" />
         <axis xyz="0 0 1" />
-        <limit lower="-1.57" upper="1.57" effort="50.0" velocity="50.0"/>
+        <limit lower="-3.14" upper="3.14" effort="50.0" velocity="50.0"/>
         <mimic joint="left_steering_hinge_joint" multiplier="-1.0" offset="0.0"/>
     </joint>

Commit message: backup with outdoor world

File: ackerman_description/urdf/fw-max.xacro (robot description, xacro)
@@ -4,13 +4,13 @@
     </link>
     <link name="base_link">
-        <visual>
-            <geometry>
-                <mesh filename="file:///home/azif/projetcs/Ackerman_ws/ackerman_description/meshes/fw-max-chassis.STL" scale="1 1 1"/>
-            </geometry>
-            <origin xyz="0.48 0.275 -0.01" rpy="1.57 0 -1.57" />
-            <material name="white">
-                <color rgba="1 1 1 1" />
-            </material>
-        </visual>
+    <visual>
+        <origin xyz="0 0 0.1" rpy="0 0 0"/>  <!-- Adjust height as needed -->
+        <geometry>
+        <box size="0.6 0.4 0.15"/>         <!-- Length, Width, Height in meters -->
+        </geometry>
+        <material name="Gray">
+        <color rgba="0.5 0.5 0.5 1.0"/>
+        </material>
+    </visual>
         <inertial>
         <origin xyz="0 0 0" />
@@ -61,5 +61,5 @@
     </transmission>
     <link name="left_front_wheel">
-        <visual><geometry><mesh filename="file:///home/azif/projetcs/Ackerman_ws/ackerman_description/meshes/fw-max-luntai.STL" scale="1 1 1"/></geometry>
+        <visual><geometry><mesh filename="file://$(find ackerman_description)/meshes/fw-max-luntai.STL" scale="1 1 1"/></geometry>
             <origin xyz="0.135 0.055 0.135" rpy="0 3.14 1.57" />
             <material name="black"><color rgba="0.0 0.0 0.0 1.0" /></material>
@@ -118,5 +118,5 @@
     </transmission>
     <link name="right_front_wheel">
-        <visual><geometry><mesh filename="file:///home/azif/projetcs/Ackerman_ws/ackerman_description/meshes/fw-max-luntai.STL" scale="1 1 1"/></geometry>
+        <visual><geometry><mesh filename="file://$(find ackerman_description)/meshes/fw-max-luntai.STL" scale="1 1 1"/></geometry>
             <origin xyz="0.135 -0.055 -0.135" rpy="0 0 1.57" />
             <material name="black"><color rgba="0.0 0.0 0.0 1.0" /></material>
@@ -174,5 +174,5 @@
     </transmission>
     <link name="left_rear_wheel">
-        <visual><geometry><mesh filename="file:///home/azif/projetcs/Ackerman_ws/ackerman_description/meshes/fw-max-luntai.STL" scale="1 1 1"/></geometry>
+        <visual><geometry><mesh filename="file://$(find ackerman_description)/meshes/fw-max-luntai.STL" scale="1 1 1"/></geometry>
             <origin xyz="0.135 0.055 0.135" rpy="0 3.14 1.57" />
             <material name="black"><color rgba="0.0 0.0 0.0 1.0" /></material>
@@ -230,5 +230,5 @@
     </transmission>
     <link name="right_rear_wheel">
-        <visual><geometry><mesh filename="file:///home/azif/projetcs/Ackerman_ws/ackerman_description/meshes/fw-max-luntai.STL" scale="1 1 1"/></geometry>
+        <visual><geometry><mesh filename="file://$(find ackerman_description)/meshes/fw-max-luntai.STL" scale="1 1 1"/></geometry>
             <origin xyz="0.135 -0.055 -0.135" rpy="0 0 1.57" />
             <material name="black"><color rgba="0.0 0.0 0.0 1.0" /></material>
